Commit message: feat: better lidar position

File: src/warehouse_bot/urdf/turtlebot3_waffle_pi.urdf (robot description, URDF)
Before this commit: robot turtlebot3_waffle_pi, 11 links, 10 joints
Joints:
- joint scan_joint: origin xyz=-0.01 0 0.122 rpy=0 0 0 -> xyz=-0.003 0 0.122 rpy=0 0 0

Commit message: feat: correct lidar position in urdf

File: src/warehouse_bot/urdf/turtlebot3_waffle_pi.urdf (robot description, URDF)
Before this commit: robot turtlebot3_waffle_pi, 11 links, 10 joints
Joints:
- joint scan_joint: origin xyz=-0.003 0 0.122 rpy=0 0 0 -> xyz=0.002 0 0.122 rpy=0 0 0
